Commit message: GitHub-ready: portable paths, docs, architecture
- Remove hardcoded /home/tech/IGVC_SIM paths from launch files
- Move Nav2 params and waypoints into orange_gazebo/config/
- Make scripts workspace-agnostic (detect from script location)
- Add docs/ (ARCHITECTURE.md, TOPIC_GRAPH.md, SETUP_GUIDE.md)
- Standardize naming to IGVC_2 in documentation
- Export IGVC_WORKSPACE in setup_orange.sh
- Works from any clone location

Made-with: Cursor

File: src/orange_ros2/orange_description/xacro/orange_robot_simulation.xacro (robot description, xacro)
@@ -31,5 +31,5 @@
     <!-- Mounted flush with pole - same height (1.0m), brought back in x -->
     <!-- Height: 1.0m, x=0.0 (flush with pole), Pitch: +0.52 rad (+30°) to see ground -->
-    <origin xyz="0.0 0.0 1.0" rpy="0.0 0.52 0.0"/>
+    <origin xyz="0.0 0.0 3.0" rpy="0.0 0.52 0.0"/>
   </xacro:oak_d_pro>
   <!--base footprint-->

File: src/orange_ros2/orange_description/xacro/sensors/oak_d_pro.xacro (robot description, xacro)
@@ -14,9 +14,9 @@
     <link name="${name}_link">
       <visual>
-        <origin xyz="0 0 0" rpy="0 0 0"/>
+        <origin xyz="0 1 3" rpy="0 0 0"/>camera
         <geometry>
           <box size="0.097 0.0275 0.0275"/>
-        </geometry>
-        <material name="oak_gray">
+        </geometry>camera
+        <material name="oak_gcameraray">
           <color rgba="0.3 0.3 0.3 1.0"/>
         </material>
