Commit message: Fix R3 sim launch and camera/perception visualization.
Align the new R3 URDF with Gazebo and RViz by cleaning up robot_description handling, stale Gazebo startup, front camera mounting, and lane debug displays so the simulated view matches the intended hardware setup.

Made-with: Cursor

File: src/orange_ros2/orange_description/URDF/urdf/r3_top_assem.xacro (robot description, xacro)
@@ -3,5 +3,5 @@
   <!-- file:// + $(find ...) so Gazebo resolves visuals when spawning URDF (package:// is unreliable). -->
   <xacro:property name="mesh_dir" value="file://$(find orange_description)/URDF/meshes"/>
-  <!-- Wheel geometry for diff_drive (meters): center-to-center along y, tire diameter -->
+  <!-- Wheel geometry for diff_drive (meters); center-to-center along y, tire diameter -->
   <xacro:property name="wheel_sep" value="0.8105"/>
   <xacro:property name="wheel_diam" value="0.44"/>
@@ -10,5 +10,5 @@
     <parent link="base_footprint"/>
     <child link="base_link"/>
-    <!-- Ground ~ wheel bottom: wheel z -0.074, r=0.22 → raise base_link ~0.29 m above footprint -->
+    <!-- Ground ~ wheel bottom; wheel z -0.074, r=0.22; raise base_link ~0.29 m above footprint -->
     <origin xyz="0 0 0.24" rpy="0 0 0"/>
   </joint>
@@ -167,5 +167,6 @@
   </xacro:sensor_imu>
   <xacro:oak_d_pro name="oak" parent="base_link">
-    <origin xyz="0.35 0 0.45" rpy="0 0.52 0"/>
+    <!-- Mounted on the front-right pole, pitched down about 20 degrees -->
+    <origin xyz="-0.31 0.0 0.81" rpy="0 0.20 0"/>
   </xacro:oak_d_pro>
   <!-- Wheel / caster friction (matches orange_robot_simulation.gazebo pattern) -->

File: src/orange_ros2/orange_description/xacro/orange_robot_simulation.xacro (robot description, xacro)
@@ -29,7 +29,6 @@
   <xacro:include filename="$(find orange_description)/xacro/sensors/oak_d_pro.xacro"/>
   <xacro:oak_d_pro name="oak" parent="base_link">
-    <!-- Mounted flush with pole - same height (1.0m), brought back in x -->
-    <!-- Height: 1.0m, x=0.0 (flush with pole), Pitch: +0.52 rad (+30°) to see ground -->
-    <origin xyz="0.0 0.0 3.0" rpy="0.0 0.52 0.0"/>
+    <!-- Mounted on the front-right pole, pitched down about 20 degrees -->
+    <origin xyz="-0.28 0.0 0.78" rpy="0.0 0.349066 0.0"/>
   </xacro:oak_d_pro>
   <!--base footprint-->

File: src/orange_ros2/orange_description/xacro/sensors/oak_d_pro.xacro (robot description, xacro)
@@ -14,8 +14,8 @@
     <link name="${name}_link">
       <visual>
-        <origin xyz="0 1 3" rpy="0 0 0"/>camera
+        <origin xyz="0 0 0" rpy="0 0 0"/>
         <geometry>
           <box size="0.097 0.0275 0.0275"/>
-        </geometry>camera
+        </geometry>
         <material name="oak_gcameraray">
           <color rgba="0.3 0.3 0.3 1.0"/>
